Commit message: add a 360 lidar and remove gazebo visu

File: tekbot/tekbot_description/urdf/tekbot.urdf (robot description, URDF)
Before this commit: robot tekbot, 4 links, 3 joints
Joints:
- joint base_joint: child base_footprint -> base_link; origin xyz=0.0 0.0 ${-(wheel_radius+wheel_zoff)} rpy=0 0 0 -> xyz=0.0 0.0 0.10 rpy=0 0 0; parent base_link -> base_footprint

Commit message: add camera

File: tekbot/tekbot_description/urdf/tekbot.urdf (robot description, URDF)
Before this commit: robot tekbot, 4 links, 3 joints
Links:
- added link camera_link; visual box size=0.02 0.02 0.02
Joints:
- added joint camera_joint: type fixed, parent base_link, child camera_link, origin xyz=0 0 0.25 rpy=0 0 0
